File: doc/Function Generator/Function Generator.sch (KiCad schematic (older format))
At the start: 30 parts, among them SW1 SW_Push, SW2 SW_Push, U1 LT1364, U2 STM8S103F3_Blue, U3 CJMCU_AD9833

Commit message: Kicad drawings
Parts:
- added C? (x2): 10u, symbol Device:C_Small
- added C?: 1000u, symbol Device:CP1_Small
Connections:
- wire segments 117 -> 126
Other:
- moved on the sheet: C8
Changed lines of the file:
@@
 L AD9833~Module:CJMCU_AD9833 U3
 U 1 1 6014CDA6
-P 4750 3350
-F 0 "U3" V 4762 3628 50  0000 L CNN
-F 1 "CJMCU_AD9833" V 4853 3628 50  0000 L CNN
-F 2 "" H 4750 3650 50  0001 C CNN
-F 3 "" H 4750 3650 50  0001 C CNN
-	1    4750 3350
+P 5550 3350
+F 0 "U3" V 5562 3628 50  0000 L CNN
+F 1 "CJMCU_AD9833" V 5653 3628 50  0000 L CNN
+F 2 "" H 5550 3650 50  0001 C CNN
+F 3 "" H 5550 3650 50  0001 C CNN
+	1    5550 3350
 	0    1    1    0
 $EndComp
@@
 $EndComp
 $Comp
-L Device:C_Small C8
-U 1 1 60156940
-P 4550 5350
-F 0 "C8" H 4642 5396 50  0000 L CNN
-F 1 "100n" H 4642 5305 50  0000 L CNN
-F 2 "" H 4550 5350 50  0001 C CNN
-F 3 "~" H 4550 5350 50  0001 C CNN
-	1    4550 5350
-	1    0    0    -1
-$EndComp
-$Comp
 L power:GND #PWR010
 U 1 1 60170584
@@
 L power:GND #PWR021
 U 1 1 60170B12
-P 4350 5600
-F 0 "#PWR021" H 4350 5350 50  0001 C CNN
-F 1 "GND" H 4355 5427 50  0000 C CNN
-F 2 "" H 4350 5600 50  0001 C CNN
-F 3 "" H 4350 5600 50  0001 C CNN
-	1    4350 5600
+P 4350 5650
+F 0 "#PWR021" H 4350 5400 50  0001 C CNN
+F 1 "GND" H 4355 5477 50  0000 C CNN
+F 2 "" H 4350 5650 50  0001 C CNN
+F 3 "" H 4350 5650 50  0001 C CNN
+	1    4350 5650
 	1    0    0    -1
 $EndComp
@@
 L power:+5V #PWR020
 U 1 1 601710DE
-P 4350 4950
-F 0 "#PWR020" H 4350 4800 50  0001 C CNN
-F 1 "+5V" H 4365 5123 50  0000 C CNN
-F 2 "" H 4350 4950 50  0001 C CNN
-F 3 "" H 4350 4950 50  0001 C CNN
-	1    4350 4950
+P 4350 4850
+F 0 "#PWR020" H 4350 4700 50  0001 C CNN
+F 1 "+5V" H 4365 5023 50  0000 C CNN
+F 2 "" H 4350 4850 50  0001 C CNN
+F 3 "" H 4350 4850 50  0001 C CNN
+	1    4350 4850
 	1    0    0    -1
 $EndComp
@@
 L power:+5V #PWR019
 U 1 1 6017A3AC
-P 4250 2800
-F 0 "#PWR019" H 4250 2650 50  0001 C CNN
-F 1 "+5V" H 4265 2973 50  0000 C CNN
-F 2 "" H 4250 2800 50  0001 C CNN
-F 3 "" H 4250 2800 50  0001 C CNN
-	1    4250 2800
+P 5050 2800
+F 0 "#PWR019" H 5050 2650 50  0001 C CNN
+F 1 "+5V" H 5065 2973 50  0000 C CNN
+F 2 "" H 5050 2800 50  0001 C CNN
+F 3 "" H 5050 2800 50  0001 C CNN
+	1    5050 2800
 	1    0    0    -1
 $EndComp
@@
 L power:GND #PWR018
 U 1 1 6017A924
-P 4000 4000
-F 0 "#PWR018" H 4000 3750 50  0001 C CNN
-F 1 "GND" H 4005 3827 50  0000 C CNN
-F 2 "" H 4000 4000 50  0001 C CNN
-F 3 "" H 4000 4000 50  0001 C CNN
-	1    4000 4000
-	1    0    0    -1
-$EndComp
-Wire Wire Line
-	4400 3250 4000 3250
-Wire Wire Line
-	4000 3250 4000 4000
-Wire Wire Line
-	4400 3150 4250 3150
-Wire Wire Line
-	4250 3150 4250 2800
-Wire Wire Line
-	4400 3350 4150 3350
-Wire Wire Line
-	4400 3450 4150 3450
-Wire Wire Line
-	4400 3550 4150 3550
-Wire Wire Line
-	4400 3650 4150 3650
-Text Label 4150 3650 0    50   ~ 0
+P 4800 4000
+F 0 "#PWR018" H 4800 3750 50  0001 C CNN
+F 1 "GND" H 4805 3827 50  0000 C CNN
+F 2 "" H 4800 4000 50  0001 C CNN
+F 3 "" H 4800 4000 50  0001 C CNN
+	1    4800 4000
+	1    0    0    -1
+$EndComp
+Wire Wire Line
+	5200 3250 4800 3250
+Wire Wire Line
+	4800 3250 4800 4000
+Wire Wire Line
+	5200 3150 5050 3150
+Wire Wire Line
+	5050 3150 5050 2800
+Wire Wire Line
+	5200 3350 4950 3350
+Wire Wire Line
+	5200 3450 4950 3450
+Wire Wire Line
+	5200 3550 4950 3550
+Wire Wire Line
+	5200 3650 4950 3650
+Text Label 4950 3650 0    50   ~ 0
 V_SIG
-Text Label 4150 3550 0    50   ~ 0
+Text Label 4950 3550 0    50   ~ 0
 SS
 Wire Wire Line
@@
 Text Label 3050 3400 0    50   ~ 0
 MOSI
-Text Label 4150 3350 0    50   ~ 0
+Text Label 4950 3350 0    50   ~ 0
 MOSI
 Text Label 3050 3500 0    50   ~ 0
 CLK
-Text Label 4150 3450 0    50   ~ 0
+Text Label 4950 3450 0    50   ~ 0
 CLK
 $Comp
@@
 FREQ_POT
 Wire Wire Line
-	4500 5250 4550 5250
-Wire Wire Line
 	4350 5100 4350 4950
 Wire Wire Line
-	4350 5400 4350 5500
-Connection ~ 4550 5250
-Wire Wire Line
-	4550 5250 4600 5250
-Wire Wire Line
-	4550 5450 4550 5500
-Wire Wire Line
-	4550 5500 4350 5500
-Connection ~ 4350 5500
-Wire Wire Line
-	4350 5500 4350 5600
+	4350 5400 4350 5550
+Connection ~ 4350 5550
+Wire Wire Line
+	4350 5550 4350 5650
 Wire Wire Line
 	1800 3800 1650 3800
@@
 Wire Wire Line
 	3900 2050 3900 2150
+$Comp
+L Device:C_Small C?
+U 1 1 6045C3E2
+P 4050 5250
+F 0 "C?" H 3850 5300 50  0000 L CNN
+F 1 "10u" H 3800 5200 50  0000 L CNN
+F 2 "" H 4050 5250 50  0001 C CNN
+F 3 "~" H 4050 5250 50  0001 C CNN
+	1    4050 5250
+	1    0    0    -1
+$EndComp
+Wire Wire Line
+	4050 5150 4050 4950
+Wire Wire Line
+	4050 4950 4350 4950
+Connection ~ 4350 4950
+Wire Wire Line
+	4350 4950 4350 4850
+Wire Wire Line
+	4050 5350 4050 5550
+Wire Wire Line
+	4050 5550 4350 5550
+$Comp
+L Device:C_Small C8
+U 1 1 60156940
+P 4600 5400
+F 0 "C8" H 4692 5446 50  0000 L CNN
+F 1 "100n" H 4692 5355 50  0000 L CNN
+F 2 "" H 4600 5400 50  0001 C CNN
+F 3 "~" H 4600 5400 50  0001 C CNN
+	1    4600 5400
+	1    0    0    -1
+$EndComp
+Wire Wire Line
+	4500 5250 4600 5250
+Wire Wire Line
+	4350 5550 4600 5550
+Wire Wire Line
+	4600 5550 4600 5500
+Wire Wire Line
+	4600 5250 4600 5300
+$Comp
+L power:+5V #PWR?
+U 1 1 604C5E89
+P 3950 3100
+F 0 "#PWR?" H 3950 2950 50  0001 C CNN
+F 1 "+5V" H 3965 3273 50  0000 C CNN
+F 2 "" H 3950 3100 50  0001 C CNN
+F 3 "" H 3950 3100 50  0001 C CNN
+	1    3950 3100
+	1    0    0    -1
+$EndComp
+$Comp
+L power:+5V #PWR?
+U 1 1 604C665E
+P 4200 3100
+F 0 "#PWR?" H 4200 2950 50  0001 C CNN
+F 1 "+5V" H 4215 3273 50  0000 C CNN
+F 2 "" H 4200 3100 50  0001 C CNN
+F 3 "" H 4200 3100 50  0001 C CNN
+	1    4200 3100
+	1    0    0    -1
+$EndComp
+$Comp
+L power:GND #PWR?
+U 1 1 604C6DC5
+P 3950 3400
+F 0 "#PWR?" H 3950 3150 50  0001 C CNN
+F 1 "GND" H 3955 3227 50  0000 C CNN
+F 2 "" H 3950 3400 50  0001 C CNN
+F 3 "" H 3950 3400 50  0001 C CNN
+	1    3950 3400
+	1    0    0    -1
+$EndComp
+$Comp
+L power:GND #PWR?
+U 1 1 604C74CC
+P 4200 3400
+F 0 "#PWR?" H 4200 3150 50  0001 C CNN
+F 1 "GND" H 4205 3227 50  0000 C CNN
+F 2 "" H 4200 3400 50  0001 C CNN
+F 3 "" H 4200 3400 50  0001 C CNN
+	1    4200 3400
+	1    0    0    -1
+$EndComp
+$Comp
+L Device:C_Small C?
+U 1 1 604C7C3B
+P 3950 3250
+F 0 "C?" H 3750 3300 50  0000 L CNN
+F 1 "10u" H 3700 3200 50  0000 L CNN
+F 2 "" H 3950 3250 50  0001 C CNN
+F 3 "~" H 3950 3250 50  0001 C CNN
+	1    3950 3250
+	1    0    0    -1
+$EndComp
+$Comp
+L Device:CP1_Small C?
+U 1 1 604E7780
+P 4200 3250
+F 0 "C?" H 4291 3296 50  0000 L CNN
+F 1 "1000u" H 4291 3205 50  0000 L CNN
+F 2 "" H 4200 3250 50  0001 C CNN
+F 3 "~" H 4200 3250 50  0001 C CNN
+	1    4200 3250
+	1    0    0    -1
+$EndComp
+Wire Wire Line
+	3950 3100 3950 3150
+Wire Wire Line
+	4200 3100 4200 3150
+Wire Wire Line
+	4200 3350 4200 3400
+Wire Wire Line
+	3950 3350 3950 3400
 $EndSCHEMATC

Commit message: tweaks to schematics
Parts:
- added L?: 10mH, symbol Device:L
Connections:
- wire segments 126 -> 128
Changed lines of the file:
@@
 L power:+5V #PWR020
 U 1 1 601710DE
-P 4350 4850
-F 0 "#PWR020" H 4350 4700 50  0001 C CNN
-F 1 "+5V" H 4365 5023 50  0000 C CNN
-F 2 "" H 4350 4850 50  0001 C CNN
-F 3 "" H 4350 4850 50  0001 C CNN
-	1    4350 4850
+P 4350 4550
+F 0 "#PWR020" H 4350 4400 50  0001 C CNN
+F 1 "+5V" H 4365 4723 50  0000 C CNN
+F 2 "" H 4350 4550 50  0001 C CNN
+F 3 "" H 4350 4550 50  0001 C CNN
+	1    4350 4550
 	1    0    0    -1
 $EndComp
@@
 Connection ~ 4350 4950
 Wire Wire Line
-	4350 4950 4350 4850
-Wire Wire Line
 	4050 5350 4050 5550
 Wire Wire Line
@@
 Wire Wire Line
 	3950 3350 3950 3400
+$Comp
+L Device:L L?
+U 1 1 60888704
+P 4350 4750
+F 0 "L?" H 4402 4796 50  0000 L CNN
+F 1 "10mH" H 4402 4705 50  0000 L CNN
+F 2 "" H 4350 4750 50  0001 C CNN
+F 3 "~" H 4350 4750 50  0001 C CNN
+	1    4350 4750
+	1    0    0    -1
+$EndComp
+Wire Wire Line
+	4350 4550 4350 4600
+Wire Wire Line
+	4350 4900 4350 4950
+Wire Wire Line
+	5550 3850 5550 4050
+Text Label 5550 4050 0    50   ~ 0
+V_SIG
 $EndSCHEMATC

Commit message: added rotary encoder to schematic
Parts:
- removed C6, C7, C8: 100n, symbol Device:C_Small
- removed C?: 10u, symbol Device:C_Small
- removed L?: 10mH, symbol Device:L
- removed R11, R8: 68, symbol Device:R_US
- removed RV3: 10k, symbol Device:R_POT_US
- removed SW1, SW2: SW_Push, symbol Switch:SW_Push
- added C? (x3): 100n, symbol Device:C_Small
- added R? (x3): 27k, symbol Device:R_US
- added SW?: Rotary_Encoder_Switch, symbol Device:Rotary_Encoder_Switch
Connections:
- net labels added: ENCODER_1, ENCODER_2, ENCODER_SW, SYSTICK
- net labels removed: SW1, SW2
- wire segments 128 -> 123

Commit message: Working, but velocity scaling needs polish
Parts:
- removed C? (x3): 100n, symbol Device:C_Small
- removed R? (x3): 27k, symbol Device:R_US
- added C? (x2): 10n, symbol Device:C_Small
- added R? (x4): 10k, symbol Device:R_US
- SW?: value Rotary_Encoder_Switch -> encoder
Connections:
- wire segments 123 -> 121
Other:
- moved on the sheet: R7

Commit message: implemented rotary encoder hardware debounce, and read inputs in an ISR
Parts:
- added C10: 10n, symbol Device:C_Small
- added R15, R16: 10k, symbol Device:R_US
- gave numbers to parts that had none: 9
Connections:
- wire segments 121 -> 131
Other:
- note added: "https://www.bourns.com/docs/technical-documents/technical-library/sensors-controls/technical-notes/Bourns_enc_sgnl_cond_technote.pdf?sfvrsn=348415eb_4"
- moved on the sheet: C6, C7, R11, R13, R14, R8
